Commit message: SLAM p1

File: description/robot_core.xacro (robot description, xacro)
@@ -6,5 +6,13 @@
     <link name="base_link">
     </link>
-    <joint name="base_link" type="fixed">
+    <joint name="base_footprint_joint" type="fixed">
+        <parent link="base_link"/>
+        <child link="base_footprint"/>
+        <origin xyz="0 0 0"/>
+    </joint>
+    <!-- Example link -->
+    <link name="base_footprint">
+    </link>
+      <joint name="base_link" type="fixed">
         <parent link="base_link"/>
         <child link="chassis"/>
